File: hw/nbiot_esp32s3_hat.kicad_pcb (KiCad board)
At the start: 2 copper layers, 65 x 30.5 mm, 79 parts, among them J1 DE9_Pins_MountingHoles, J3 USB_A, J4 Conn_02x20_Odd_Even, J5 USB_C_Receptacle_USB2.0_16P, Q1 SS8050, Q2 SS8050, U1 TP5100, U2 AMS1117-3.3, U3 ESP32-S3-MINI-1U, U4 CH343P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

Commit message: hw: further work on PCB
Parts:
- added C23: C, Capacitor_SMD:C_0603_1608Metric, F.Cu at (93.6, -42.1)
- added C24: 33pF, Capacitor_SMD:C_0402_1005Metric, F.Cu at (104.3, -42.8)
- added C25: 33pF, Capacitor_SMD:C_0402_1005Metric, F.Cu at (104.3, -40.8)
- added C26: 33pF, Capacitor_SMD:C_0402_1005Metric, F.Cu at (104.3, -38.9)
- added C27: C, Capacitor_SMD:C_0603_1608Metric, F.Cu at (93.6, -39.6)
- added C28: C, Capacitor_SMD:C_0603_1608Metric, F.Cu at (93.6, -37.0)
- added C31: 100n, Capacitor_SMD:C_0402_1005Metric, F.Cu at (104.3, -36.9)
- added C36: 10u, Capacitor_SMD:C_0805_2012Metric, F.Cu at (93.8, -34.3)
- added C37: 10u, Capacitor_SMD:C_0805_2012Metric, F.Cu at (93.8, -31.3)
- added D6: LED, LED_SMD:LED_0603_1608Metric, F.Cu at (107.8, -37.9)
- added J2: SIM_Card, Connector_Card:nanoSIM_Hinged_CUI_NSIM-2-C, F.Cu at (121.8, -21.2)
- added Q3: SS8050, Package_TO_SOT_SMD:SOT-23, F.Cu at (94.1, -50.0)
- added Q5: SS8050, Package_TO_SOT_SMD:SOT-23, F.Cu at (94.1, -45.5)
- added R26: 4,7K, Resistor_SMD:R_0402_1005Metric, F.Cu at (78.0, -34.8)
- added R27: 100R, Resistor_SMD:R_0402_1005Metric, F.Cu at (78.0, -32.8)
- added R28: 22, Resistor_SMD:R_0402_1005Metric, F.Cu at (78.0, -30.8)
- added R29: 22, Resistor_SMD:R_0402_1005Metric, F.Cu at (80.9, -34.8)
- added R30: 22, Resistor_SMD:R_0402_1005Metric, F.Cu at (80.9, -32.8)
- added R31: R, Resistor_SMD:R_0402_1005Metric, F.Cu at (80.9, -30.8)
- added R32: R, Resistor_SMD:R_0402_1005Metric, F.Cu at (83.8, -34.8)
- added R33: 4,7K, Resistor_SMD:R_0402_1005Metric, F.Cu at (83.8, -32.8)
- added R34: 47K, Resistor_SMD:R_0402_1005Metric, F.Cu at (83.8, -30.8)
- added SW1: SW_Push, Button_Switch_SMD:SW_SPST_TS-1088-xR020, F.Cu at (110.5, -44.5)
- R12: value 100k -> 47K
Connections:
- net Net-(U7-VBAT-Pad34) renamed VBAT
- R12 pad 1: BOOST_EN -> Net-(Q3-B)
- U7 pad 13: Net-(U7-GND-Pad13) -> GND
- U7 pad 19: Net-(U7-GND-Pad13) -> GND
- U7 pad 20: unconnected-(U7-IO_1833_SEL-Pad20) -> GND
- U7 pad 21: Net-(U7-GND-Pad13) -> GND
- U7 pad 22: unconnected-(U7-UART0_TXD-Pad22) -> NBIOT_RX
- U7 pad 23: unconnected-(U7-UART0_RXD-Pad23) -> NBIOT_TX
- U7 pad 27: Net-(U7-GND-Pad13) -> GND
- U7 pad 28: unconnected-(U7-~{RESET}-Pad28) -> NB_RST
- U7 pad 30: Net-(U7-GND-Pad13) -> GND
- U7 pad 31: Net-(U7-GND-Pad13) -> GND
- U7 pad 32: unconnected-(U7-ANT-Pad32) -> RF_ANT
- U7 pad 33: Net-(U7-GND-Pad13) -> GND
- U7 pad 36: Net-(U7-GND-Pad13) -> GND
- U7 pad 37: Net-(U7-GND-Pad13) -> GND
- U7 pad 41: unconnected-(U7-NETLIGHT-Pad41) -> NETLIGHT
- U7 pad 8: Net-(U7-GND-Pad13) -> GND
Routing:
- net BOOST_EN: track 34.0 -> 0.00 mm
- net (no net): track 0.00 -> 34.0 mm
Other:
- board size 65 x 30.5 mm -> 100 x 134.6 mm
