File: hw/nbiot_esp32s3_hat.kicad_sch (KiCad schematic)
At the start: 103 parts, among them J1 DE9_Pins_MountingHoles, J2 SIM_Card, J3 USB_A, J5 USB_C_Receptacle_USB2.0_16P, Q1 SS8050, Q2 SS8050, Q3 MMBT3904, Q4 MMBT3904, SW1 SW_Push, U1 TP5100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

Commit message: hw: further work on PCB
Parts:
- removed C29: 10uF, symbol Device:C
- removed C30: C, symbol Device:C
- removed D7: B5819WS-TP, B5819WS-TP:SOD2512X115N, symbol kolskypavel:B5819WS-TP
- removed Q3, Q4: MMBT3904, Package_TO_SOT_SMD:SOT-23, symbol Transistor_BJT:MMBT3904
- removed U8: TVS0500DRV, Package_SON:WSON-6-1EP_2x2mm_P0.65mm_EP1x1.6mm, symbol Power_Protection:TVS0500DRV
- added C36, C37: 10u, Capacitor_SMD:C_0805_2012Metric, symbol Device:C
- added Q3, Q5: SS8050, Package_TO_SOT_SMD:SOT-23, symbol Transistor_BJT:SS8050
- C23, C27, C28: footprint (none) -> Capacitor_SMD:C_0603_1608Metric
- C24, C25, C26: footprint (none) -> Capacitor_SMD:C_0402_1005Metric
- C31: value 104 -> 100n; footprint (none) -> Capacitor_SMD:C_0402_1005Metric
- D6: footprint (none) -> LED_SMD:LED_0603_1608Metric
- J2: footprint (none) -> Connector_Card:nanoSIM_Hinged_CUI_NSIM-2-C
- R12, R26, R28, R29, R30, R31, R32, R33, R34: footprint (none) -> Resistor_SMD:R_0402_1005Metric
- R27: value ~ -> 100R; footprint (none) -> Resistor_SMD:R_0402_1005Metric
- SW1: footprint (none) -> Button_Switch_SMD:SW_SPST_TS-1088-xR020
Connections:
- net +3.3V: now also D6.2 (A); no longer U7.34 (VBAT), U7.35 (VBAT)
- net GND: now also C36.2, C37.2, Q3.2 (E), Q5.2 (E)
- net at R12.1, R26.2: now also Q3.1 (B)
- net at R27.1: now also Q3.3 (C)
- net at R33.2, R34.1: now also Q5.1 (B)
- net at C31.1, SW1.1: now also Q5.3 (C)
- new net VBAT: C36.1, C37.1, U7.34 (VBAT), U7.35 (VBAT)
