File: hw/oracon/oracon.kicad_sch (KiCad schematic)
At the start: 104 parts, among them J2 SIM_Holder, J3 USB_A, J4 Conn_Coaxial, J5 USB_C_Receptacle_USB2.0_16P, J6 Conn_01x02_MountingPin, Q1 SS8050, Q2 SS8050, Q3 SS8050, SW3 SW_Push, U1 TP5100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

Commit message: To be checked for production.
Parts:
- J6: footprint (none) -> kolskypavel:CONN-TH_B2B-PH-K-S; lcsc (none) -> C131337
Connections:
- net USB_SI_N: now also U3.23 (IO19); no longer U3.7 (IO3)
- net USB_SI_P: now also U3.24 (IO20); no longer U3.8 (IO4)
Changed lines of the file:
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@@
 		)
 	)
-	(global_label "USB_SI_N"
-		(shape input)
-		(at 48.26 109.22 180)
-		(fields_autoplaced yes)
-		(effects
-			(font
-				(size 1.27 1.27)
-			)
-			(justify right)
-		)
-		(property "Intersheetrefs" "${INTERSHEET_REFS}"
-			(at 36.3848 109.22 0)
-			(effects
-				(font
-					(size 1.27 1.27)
-				)
-				(justify right)
-				(hide yes)
-			)
-		)
-	)
 	(global_label "NBIOT_TX"
 		(shape input)
@@
 		)
 	)
+	(global_label "USB_SI_N"
+		(shape input)
+		(at 80.01 104.14 0)
+		(fields_autoplaced yes)
+		(effects
+			(font
+				(size 1.27 1.27)
+			)
+			(justify left)
+		)
+		(property "Intersheetrefs" "${INTERSHEET_REFS}"
+			(at 91.8852 104.14 0)
+			(effects
+				(font
+					(size 1.27 1.27)
+				)
+				(justify left)
+				(hide yes)
+			)
+		)
+	)
 	(global_label "LED1_G"
 		(shape input)
@@
 		)
 	)
-	(global_label "USB_SI_P"
+	(global_label "STBY_STAT"
 		(shape input)
-		(at 48.26 111.76 180)
+		(at 375.92 111.76 180)
 		(fields_autoplaced yes)
 		(effects
@@
 		)
 		(property "Intersheetrefs" "${INTERSHEET_REFS}"
-			(at 36.4453 111.76 0)
+			(at 363.1982 111.76 0)
 			(effects
 				(font
@@
 		)
 	)
-	(global_label "STBY_STAT"
+	(global_label "USB_SI_N"
 		(shape input)
-		(at 375.92 111.76 180)
+		(at 384.81 165.1 0)
 		(fields_autoplaced yes)
 		(effects
@@
 				(size 1.27 1.27)
 			)
-			(justify right)
+			(justify left)
 		)
 		(property "Intersheetrefs" "${INTERSHEET_REFS}"
-			(at 363.1982 111.76 0)
+			(at 396.6852 165.1 0)
 			(effects
 				(font
 					(size 1.27 1.27)
 				)
-				(justify right)
+				(justify left)
 				(hide yes)
 			)
 		)
 	)
-	(global_label "USB_SI_N"
+	(global_label "RS232_TX"
 		(shape input)
-		(at 384.81 165.1 0)
+		(at 48.26 104.14 180)
 		(fields_autoplaced yes)
 		(effects
@@
 				(size 1.27 1.27)
 			)
-			(justify left)
+			(justify right)
 		)
 		(property "Intersheetrefs" "${INTERSHEET_REFS}"
-			(at 396.6852 165.1 0)
+			(at 36.0221 104.14 0)
 			(effects
 				(font
 					(size 1.27 1.27)
 				)
-				(justify left)
+				(justify right)
 				(hide yes)
 			)
 		)
 	)
-	(global_label "RS232_TX"
+	(global_label "USB_SI_P"
 		(shape input)
-		(at 48.26 104.14 180)
+		(at 80.01 106.68 0)
 		(fields_autoplaced yes)
 		(effects
@@
 				(size 1.27 1.27)
 			)
-			(justify right)
+			(justify left)
 		)
 		(property "Intersheetrefs" "${INTERSHEET_REFS}"
-			(at 36.0221 104.14 0)
+			(at 91.8247 106.68 0)
 			(effects
 				(font
 					(size 1.27 1.27)
 				)
-				(justify right)
+				(justify left)
 				(hide yes)
 			)
@@
 			)
 		)
-		(property "Footprint" ""
+		(property "Footprint" "kolskypavel:CONN-TH_B2B-PH-K-S"
 			(at 226.06 39.37 0)
 			(effects
@@
 			(at 226.06 39.37 0)
 			(effects
+				(font
+					(size 1.27 1.27)
+				)
+				(hide yes)
+			)
+		)
+		(property "lcsc" "C131337"
+			(at 226.06 39.37 0)
+			(effects

Commit message: added connectors, USB + dimensions to be checked
Parts:
- removed C14: 10u, Capacitor_SMD:C_0805_2012Metric, symbol Device:C
- removed H5: SI_TX, TestPoint:TestPoint_Pad_D1.5mm, symbol Mechanical:MountingHole_Pad
- removed H6: SI_RX, TestPoint:TestPoint_Pad_D1.5mm, symbol Mechanical:MountingHole_Pad
- removed H7: SI_GND, TestPoint:TestPoint_Pad_D1.5mm, symbol Mechanical:MountingHole_Pad
- removed H8: SI_3.3V, TestPoint:TestPoint_Pad_D1.5mm, symbol Mechanical:MountingHole_Pad
- removed TP3: SW1, TestPoint:TestPoint_Pad_D1.5mm, symbol Connector:TestPoint
- removed TP4: SW2, TestPoint:TestPoint_Pad_D1.5mm, symbol Connector:TestPoint
- removed TP5: Serial_TX, TestPoint:TestPoint_Pad_D1.5mm, symbol Connector:TestPoint
- removed TP6: Serial_RX, TestPoint:TestPoint_Pad_D1.5mm, symbol Connector:TestPoint
- removed TP7: Serial_GND, TestPoint:TestPoint_Pad_D1.5mm, symbol Connector:TestPoint
- added C29: 100n, Capacitor_SMD:C_0402_1005Metric, symbol Device:C
- added CN1: B3B-PH-K-S, kolskypavel:CONN-TH_B3B-PH-K-S, symbol kolskypavel:B3B-PH-K-S
- added J1: Conn_01x02_MountingPin, kolskypavel:CONN-TH_B2B-PH-K-S, symbol Connector_Generic_MountingPin:Conn_01x02_MountingPin
- added U8: B4B-XH-A, kolskypavel:CONN-TH_B04B-PASK-1-LF-SN, symbol kolskypavel:B4B-XH-A
Connections:
- net +3.3V: now also U8.1
- net +BATT: now also J1.2 (Pin_2)
- net GND: now also C29.2, CN1.3, J1.MP (MountPin), U8.2
- net RST: now also C29.1
- net SI_RX: now also U8.4
- net SI_TX: now also U8.3
- net VCC: now also J1.1 (Pin_1)
- net at U6.13 (R1IN): now also CN1.2
- net at U6.14 (T1OUT): now also CN1.1
Other:
- note added: "RX"
- note added: "TX"
- company: kolskypavel -> Pavel Kolský
