File: hw/oracon/oracon.kicad_sch (KiCad schematic)
At the start: 98 parts, among them CN1 B3B-PH-K-S, J1 Conn_01x02_MountingPin, J2 SIM_Holder, J3 USB_A, J4 Conn_Coaxial, J5 USB_C_Receptacle_USB2.0_16P, J6 Conn_01x02_MountingPin, Q1 SS8050, Q2 SS8050, Q3 SS8050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

Commit message: usb position modifications
Parts:
- U8: value B4B-XH-A -> B4B-PH-K-S; footprint kolskypavel:CONN-TH_B04B-PASK-1-LF-SN -> kolskypavel:CONN-TH_B4B-PH-K-S; LCSC Part C144395 -> C131334; MPN B4B-XH-A(LF)(SN) -> B4B-PH-K-S(LF)(SN)
Changed lines of the file:
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@@
 			)
 		)
-		(property "Value" "B4B-XH-A"
+		(property "Value" "B4B-PH-K-S"
 			(at 128.27 140.9699 0)
 			(effects
@@
 			)
 		)
-		(property "Footprint" "kolskypavel:CONN-TH_B04B-PASK-1-LF-SN"
+		(property "Footprint" "kolskypavel:CONN-TH_B4B-PH-K-S"
 			(at 120.65 151.13 0)
 			(effects
@@
 			)
 		)
-		(property "Datasheet" "https://lcsc.com/product-detail/_JST-Sales-America_B4B-XH-A-LF-SN_JST-Sales-America-B4B-XH-A-LF-SN_C144395.html"
+		(property "Datasheet" ""
 			(at 120.65 153.67 0)
 			(effects
@@
 			)
 		)
-		(property "MPN" "B4B-XH-A(LF)(SN)"
+		(property "MPN" "B4B-PH-K-S(LF)(SN)"
 			(at 120.65 158.75 0)
 			(effects
@@
 			)
 		)
-		(property "LCSC Part" "C144395"
+		(property "LCSC Part" "C131334"
 			(at 120.65 161.29 0)
 			(effects
